File: Kicad/dram.sch (KiCad schematic (older format))
At the start: 8 parts, among them U45 74ABT16245, U46 74ABT16245, U47 74ABT16245, U48 74ABT16245, U49 SN74AS258, U50 SN74AS258

Commit message: some more dram
Parts:
- added CN13, CN14, CN15, CN16: GVP_SIMM, symbol New_Library_0:GVP_SIMM
- added RP15: R_Pack04_SIP, Resistor_THT:R_Array_SIP8, symbol Device:R_Pack04_SIP
- gave numbers to parts that had none: 1
Connections:
- net DRA_A4A5: now reaches U49.4 (Y1)
- net DRA_A6A7: now reaches U49.7 (Y2)
- net D_A4A5: now reaches RP23.1 (R1.1)
- net D_A4A5: now also RP23.2 (R1.2)
- net D30: now reaches U48.11 (B6)
- net D30: now also U46.11 (B6)
- net D31: now reaches U48.12 (B7)
- net D31: now also U46.12 (B7)
- net D16: now reaches U48.13 (B8)
- net D16: now also U46.13 (B8)
- net D17: now reaches U48.14 (B9)
- net D17: now also U46.14 (B9)
- net D18: now reaches U48.16 (B10)
- net D18: now also U46.16 (B10)
- net D19: now reaches U48.17 (B11)
- net D19: now also U46.17 (B11)
- net D20: now reaches U48.19 (B12)
- net D20: now also U46.19 (B12)
- net D24: now reaches U48.2 (B0)
- net D24: now also U46.2 (B0)
- net D21: now reaches U48.20 (B13)
- net D21: now also U46.20 (B13)
- net D22: now reaches U48.22 (B14)
- net D22: now also U46.22 (B14)
- net D23: now reaches U48.23 (B15)
- net D23: now also U46.23 (B15)
- net at U48.25 (_OE2): now also U47.25 (_OE2)
- net DRD23: now reaches U48.26 (A15)
- net DRD23: now also U46.26 (A15)
- net DRD22: now reaches U48.27 (A14)
- net DRD22: now also U46.27 (A14)
- net DRD21: now reaches U48.29 (A13)
- net DRD21: now also U46.29 (A13)
- net D25: now reaches U48.3 (B1)
- net D25: now also U46.3 (B1)
- net DRD20: now reaches U48.30 (A12)
- net DRD20: now also U46.30 (A12)
- net DRD19: now reaches U48.32 (A11)
- net DRD19: now also U46.32 (A11)
- net DRD18: now reaches U48.33 (A10)
- net DRD18: now also U46.33 (A10)
- net DRD17: now reaches U48.35 (A9)
- net DRD17: now also U46.35 (A9)
- net DRD16: now reaches U48.36 (A8)
- net DRD16: now also U46.36 (A8)
- net DRD31: now reaches U48.37 (A7)
- net DRD31: now also U46.37 (A7)
- net DRD30: now reaches U48.38 (A6)
- net DRD30: now also U46.38 (A6)
- net DRD29: now reaches U48.40 (A5)
- net DRD29: now also U46.40 (A5)
- net DRD28: now reaches U48.41 (A4)
- net DRD28: now also U46.41 (A4)
- net DRD27: now reaches U48.43 (A3)
- net DRD27: now also U46.43 (A3)
- net DRD26: now reaches U48.44 (A2)
- net DRD26: now also U46.44 (A2)
- net DRD25: now reaches U48.46 (A1)
- net DRD25: now also U46.46 (A1)
- net DRD24: now reaches U48.47 (A0)
- net DRD24: now also U46.47 (A0)
- net at U48.48 (_OE1): now also U47.48 (_OE1)
- net D26: now reaches U48.5 (B2)
- net D26: now also U46.5 (B2)
- net D27: now reaches U48.6 (B3)
- net D27: now also U46.6 (B3)
- net D28: now reaches U48.8 (B4)
- net D28: now also U46.8 (B4)
- net D29: now reaches U48.9 (B5)
- net D29: now also U46.9 (B5)
- net D14: now reaches U47.11 (B6)
- net D15: now reaches U47.12 (B7)
- net D15: now also U45.12 (B7)
- net D0: now reaches U47.13 (B8)
- net D0: now also U45.13 (B8)
- net D1: now reaches U47.14 (B9)
- net D2: now reaches U47.16 (B10)
- net D3: now reaches U47.17 (B11)
- net D4: now reaches U47.19 (B12)
- net D8: now reaches U47.2 (B0)
- net D8: now also U45.2 (B0)
- net D5: now reaches U47.20 (B13)
- net D6: now reaches U47.22 (B14)
- net D7: now reaches U47.23 (B15)
- net D7: now also U45.23 (B15)
- net DRD7: now reaches U47.26 (A15)
- net DRD7: now also U45.26 (A15)
- net DRD6: now reaches U47.27 (A14)
- net DRD6: now also U45.27 (A14)
- net DRD5: now reaches U47.29 (A13)
- net DRD5: now also U45.29 (A13)
- net D9: now reaches U47.3 (B1)
- net DRD4: now reaches U47.30 (A12)
- net DRD4: now also U45.30 (A12)
- net DRD3: now reaches U47.32 (A11)
- net DRD3: now also U45.32 (A11)
- net DRD2: now reaches U47.33 (A10)
- net DRD2: now also U45.33 (A10)
- net DRD1: now reaches U47.35 (A9)
- net DRD1: now also U45.35 (A9)
- net DRD0: now reaches U47.36 (A8)
- net DRD0: now also U45.36 (A8)
- net DRD15: now reaches U47.37 (A7)
- net DRD15: now also U45.37 (A7)
- net DRD14: now reaches U47.38 (A6)
- net DRD14: now also U45.38 (A6)
- net DRD13: now reaches U47.40 (A5)
- net DRD13: now also U45.40 (A5)
- net DRD12: now reaches U47.41 (A4)
- net DRD12: now also U45.41 (A4)
- net DRD11: now reaches U47.43 (A3)
- net DRD11: now also U45.43 (A3)
- net DRD10: now reaches U47.44 (A2)
- net DRD10: now also U45.44 (A2)
- net DRD9: now reaches U47.46 (A1)
- net DRD9: now also U45.46 (A1)
- net DRD8: now reaches U47.47 (A0)
- net DRD8: now also U45.47 (A0)
- net D10: now reaches U47.5 (B2)
- net D11: now reaches U47.6 (B3)
- net D12: now reaches U47.8 (B4)
- net D13: now reaches U47.9 (B5)
- net at U46.25 (_OE2): now also U45.25 (_OE2)
- net at U46.48 (_OE1): now also U45.48 (_OE1)
- new net U44_19: RP15.3 (R2.1)
Other:
- moved on the sheet: RP23, RP24, U45, U46, U48

Commit message: Some more work on dram
Parts:
- added RP16, RP17, RP18, RP19, RP20, RP21, RP22: 33R, Resistor_THT:R_Array_SIP8, symbol Device:R_Pack04_SIP
- RP15, RP23, RP24: value R_Pack04_SIP -> 33R
Connections:
- net labels added: CAS_B0, CAS_B1, CAS_B2, CAS_B3, DRA_???_DRAM_A???, DRA_A8A9, U38_15, U38_22, U39_17, U39_18, U39_19, U39_20, U40_18, U40_22, U41_17, U41_18, U41_21, U41_22, U42_15, U42_16, U42_17, U42_18, U42_22, U44_22, _CAS_B0, _CAS_B1, _CAS_B2, _CAS_B3, _OE_B0, _OE_B1, _OE_B2, _OE_B3, _RAS_B0, _RAS_B1, _RAS_B2, _RAS_B3, _WE1_B0, _WE1_B1, _WE1_B2, _WE1_B3, _WE2_B0, _WE2_B1
- wire segments 234 -> 429
Other:
- moved on the sheet: CN13, CN14, CN15, CN16

Commit message: amother day, another tracks..
Parts:
- removed RP15, RP16, RP17, RP18, RP19, RP20, RP21, RP22, RP23, RP24: 33R, Resistor_THT:R_Array_SIP8, symbol Device:R_Pack04_SIP
- added RP15, RP16, RP17, RP18, RP19, RP20, RP21, RP22, RP23, RP24: 33R, symbol New_Library_0:RPACK_04
- added U38, U39, U40, U41: PALCE20V8H_DIL, symbol New_Library_0:PALCE20V8H_DIL
- added U42, U44: PAL20L8, symbol Logic_Programmable:PAL20L8
- added U51: DM74AS74M, symbol New_Library_0:DM74AS74M
- CN13: value GVP_SIMM -> BANK_0
- CN14: value GVP_SIMM -> BANK_1
- CN15: value GVP_SIMM -> BANK_2
- CN16: value GVP_SIMM -> BANK_3
Connections:
- net labels added: DA_12_13, DA_14_15, DA_16_17, DA_18_19, U2_1, U30_18, U38_11, U38_14, U39_15, U39_22, U3_11, U40_14, U42_11, U46_20, U48_20, U51_4, U6_73, _CLK, _WE2_B2, _WE2_B3, _WE3_B0, _WE3_B1, _WE3_B2, _WE3_B3, _WE4_B0, _WE4_B1, _WE4_B2, _WE4_B3
- net labels removed: CAS_B0, DRA_BUS, U39_17, U39_18, U39_19, U40_18, U40_22, U41_17, U41_18, U41_21, U41_22, U42_15, U42_16, U42_17, U42_18, U42_22
- wire segments 429 -> 533
Other:
- moved on the sheet: CN13, CN14, CN15, CN16
